File: faceplates/C64 Joykey Faceplate B1/C64 Joykey Faceplate B1.sch (KiCad schematic (older format))
At the start: 4 parts, among them M1 Mounting, M2 Mounting, M3 Mounting, M4 Mounting

Commit message: Moved faceplates into separate folder.
Parts:
- M1, M2, M3, M4: symbol mounting:Mounting -> Connector:Conn_01x01_Male
Connections:
- wire segments 0 -> 7
Changed lines of the file:
@@
 encoding utf-8
 Sheet 1 1
-Title "C64 Joykey (Faceplate)"
+Title "C64 Joykey (Faceplate B)"
 Date ""
 Rev "A"
@@
 Comment1 ""
 Comment2 ""
-Comment3 ""
+Comment3 "This was designed for keycaps that don't go down past the top of the switches."
 Comment4 "It's just a faceplate, nothing to see here."
 $EndDescr
 $Comp
-L mounting:Mounting M1
+L Connector:Conn_01x01_Male M1
 U 1 1 5FB6F935
 P 10700 550
@@
 F 3 "~" H 10700 550 50  0001 C CNN
 	1    10700 550
-	1    0    0    -1
+	0    1    1    0
 $EndComp
 $Comp
-L mounting:Mounting M2
+L Connector:Conn_01x01_Male M2
 U 1 1 5FB70096
 P 10825 550
@@
 F 3 "~" H 10825 550 50  0001 C CNN
 	1    10825 550
-	1    0    0    -1
+	0    1    1    0
 $EndComp
 $Comp
-L mounting:Mounting M3
+L Connector:Conn_01x01_Male M3
 U 1 1 5FB70244
 P 10975 550
@@
 F 3 "~" H 10975 550 50  0001 C CNN
 	1    10975 550
-	1    0    0    -1
+	0    1    1    0
 $EndComp
 $Comp
-L mounting:Mounting M4
+L Connector:Conn_01x01_Male M4
 U 1 1 5FB705F7
 P 11100 550
@@
 F 3 "~" H 11100 550 50  0001 C CNN
 	1    11100 550
-	1    0    0    -1
+	0    1    1    0
 $EndComp
+Wire Wire Line
+	10700 750  10700 825
+Wire Wire Line
+	10700 825  10825 825
+Wire Wire Line
+	11100 825  11100 750
+Wire Wire Line
+	10975 750  10975 825
+Connection ~ 10975 825
+Wire Wire Line
+	10975 825  11100 825
+Wire Wire Line
+	10825 750  10825 825
+Connection ~ 10825 825
+Wire Wire Line
+	10825 825  10975 825
 $EndSCHEMATC
