File: adapters/IDC to DB9/IDC to DB9.sch (KiCad schematic (older format))
At the start: 2 parts, among them J1 JoyKEY, J2 DB9

Commit message: Added VCC_EN to IDC -> DB9 adapter
Parts:
- added JP1: VCC_EN, solder_bridge:bridge, symbol Device:Jumper_NC_Small
Connections:
- net VCC: now also JP1.2; no longer J1.7 (Pin_7)
- new net: J1.7 (Pin_7), JP1.1
Other:
- note added: "A straight 2x5 pin IDC to DB9 adapter, this should allow the C64 JoyKEY to connect to systems where\nthe case shape normally would conflict with the IDC DB9 connectors. Link VCC_EN if you want to allow\ndevice to supply power to port."
- note removed: "A straight 2x5 pin IDC to DB9 adapter, this should allow the C64 JoyKEY to connect to systems where\nthe case shape normally would conflict with the IDC DB9 connectors."
Changed lines of the file:
@@
 	1    0    0    -1
 $EndComp
-Text Notes 7000 6725 0    50   ~ 0
-A straight 2x5 pin IDC to DB9 adapter, this should allow the C64 JoyKEY to connect to systems where\nthe case shape normally would conflict with the IDC DB9 connectors.
+Text Notes 7000 6800 0    50   ~ 0
+A straight 2x5 pin IDC to DB9 adapter, this should allow the C64 JoyKEY to connect to systems where\nthe case shape normally would conflict with the IDC DB9 connectors. Link VCC_EN if you want to allow\ndevice to supply power to port.
 $Comp
 L joykey_jumpers:JUMPER_SETTINGS_1 #1
@@
 L power:VCC #PWR0102
 U 1 1 60066CE7
-P 4325 2225
-F 0 "#PWR0102" H 4325 2075 50  0001 C CNN
-F 1 "VCC" H 4340 2398 50  0000 C CNN
-F 2 "" H 4325 2225 50  0001 C CNN
-F 3 "" H 4325 2225 50  0001 C CNN
-	1    4325 2225
+P 4325 2025
+F 0 "#PWR0102" H 4325 1875 50  0001 C CNN
+F 1 "VCC" H 4340 2198 50  0000 C CNN
+F 2 "" H 4325 2025 50  0001 C CNN
+F 3 "" H 4325 2025 50  0001 C CNN
+	1    4325 2025
 	1    0    0    -1
 $EndComp
@@
 Wire Wire Line
 	6975 4050 6975 4650
+$Comp
+L Device:Jumper_NC_Small JP1
+U 1 1 600B5A02
+P 4325 2125
+F 0 "JP1" H 4325 2337 50  0000 C CNN
+F 1 "VCC_EN" H 4325 2246 50  0000 C CNN
+F 2 "solder_bridge:bridge" H 4325 2125 50  0001 C CNN
+F 3 "~" H 4325 2125 50  0001 C CNN
+	1    4325 2125
+	0    -1   -1   0
+$EndComp
 $EndSCHEMATC
