File: adapters/Sega Mega Drive/Sega Mega Drive.kicad_pcb (KiCad board)
At the start: 2 copper layers, 58.4 x 38.1 mm, 20 parts, among them J1 Port 1, J2 Port 2, J3 Sega Mega Drive, J4 START_SEL, M1 Mounting, M2 Mounting, M3 Mounting, M4 Mounting, SW1 START, U1 74LS157

Commit message: Exported SMD alpha
Parts:
- added R9: 10k, Resistor_THT:R_Axial_DIN0207_L6.3mm_D2.5mm_P10.16mm_Horizontal, F.Cu at (128.3, 88.9)
- R1, R2, R3, R4, R5, R6, R7, R8: value R -> 10k
- moved JP1 2.54 mm to (170.2, 95.9)
Routing:
- net /MD_SEL: track 18.6 -> 55.1 mm, vias 0 -> 1
- net /JK_START: track 68.0 -> 76.1 mm
- net VCC: track 107.8 -> 111.1 mm
- net /JK_FIRE2: track 23.3 -> 21.8 mm
- net Net-(J2-Pad7): track 29.1 -> 28.2 mm
Other:
- board text added: "(PORT 1)"
- board text added: "FIRE1"
- board text added: "FIRE2"
- board text added: "FIRE3"
- board text added: "J4 START_SEL"
- board text added: "JP1 VCC_EN"
- board text added: "P1 FIRE 1"
- board text added: "Sega Mega Drive/Genesis (C64 JoyKEY Adapter) github.com/tebl"
- board text removed: "P1 FIRE1"
- board text removed: "P1 FIRE2"
- board text removed: "P1 FIRE3"
- board text removed: "Sega Mega Drive Adapter (C64 JoyKEY) github.com/tebl"
