File: adapters/Sega Mega Drive/Sega Mega Drive.sch (KiCad schematic (older format))
At the start: 20 parts, among them J1 Port 1, J2 Port 2, J3 Sega Mega Drive, J4 START_SEL, M1 Mounting, M2 Mounting, M3 Mounting, M4 Mounting, SW1 START, U1 74LS157

Commit message: Exported SMD alpha
Parts:
- added R9: 10k, Resistor_THT:R_Axial_DIN0207_L6.3mm_D2.5mm_P10.16mm_Horizontal, symbol Device:R
- R1, R2, R3, R4, R5, R6, R7, R8: value R -> 10k
Connections:
- net MD_SEL: now also R9.2
- net VCC: now also R9.1
Other:
- note added: "Transforms the C64 JoyKEY into a simple 3-button controller for the Sega Mega Drive (named Sega\nGenesis in North America). Given that we are missing one of the buttons, this adapter has a separate\nSTART button when used with the base unit (C64 Arcade version can assign any of the other 3 buttons to\nthis).\n\nThis design is untested!"
- note removed: "Need to check what the\nresistors needs to be."
- note removed: "Transforms the C64 JoyKEY into a simple 3-button controller for the Sega Mega Drive (named Sega\nGenesis in North America). Given that we are missing one of the buttons, this adapter has a separate\nSTART button when used with the base unit (C64 Arcade version can assign any of the other 3 buttons to\nthis)."
Changed lines of the file:
@@
 	1    0    0    -1
 $EndComp
-Text Notes 7000 6900 0    50   ~ 0
-Transforms the C64 JoyKEY into a simple 3-button controller for the Sega Mega Drive (named Sega\nGenesis in North America). Given that we are missing one of the buttons, this adapter has a separate\nSTART button when used with the base unit (C64 Arcade version can assign any of the other 3 buttons to\nthis).
+Text Notes 7000 7050 0    50   ~ 0
+Transforms the C64 JoyKEY into a simple 3-button controller for the Sega Mega Drive (named Sega\nGenesis in North America). Given that we are missing one of the buttons, this adapter has a separate\nSTART button when used with the base unit (C64 Arcade version can assign any of the other 3 buttons to\nthis).\n\nThis design is untested!
 $Comp
 L mounting:Mounting M1
@@
 P 4975 2650
 F 0 "R1" V 4925 2400 50  0000 L CNN
-F 1 "R" V 4975 2625 50  0000 L CNN
+F 1 "10k" V 4975 2575 50  0000 L CNN
 F 2 "Resistor_THT:R_Axial_DIN0207_L6.3mm_D2.5mm_P10.16mm_Horizontal" V 4905 2650 50  0001 C CNN
 F 3 "~" H 4975 2650 50  0001 C CNN
@@
 P 5075 2650
 F 0 "R2" V 5025 2400 50  0000 L CNN
-F 1 "R" V 5075 2625 50  0000 L CNN
+F 1 "10k" V 5075 2575 50  0000 L CNN
 F 2 "Resistor_THT:R_Axial_DIN0207_L6.3mm_D2.5mm_P10.16mm_Horizontal" V 5005 2650 50  0001 C CNN
 F 3 "~" H 5075 2650 50  0001 C CNN
@@
 P 5175 2650
 F 0 "R3" V 5125 2400 50  0000 L CNN
-F 1 "R" V 5175 2625 50  0000 L CNN
+F 1 "10k" V 5175 2575 50  0000 L CNN
 F 2 "Resistor_THT:R_Axial_DIN0207_L6.3mm_D2.5mm_P10.16mm_Horizontal" V 5105 2650 50  0001 C CNN
 F 3 "~" H 5175 2650 50  0001 C CNN
@@
 P 5275 2650
 F 0 "R4" V 5225 2400 50  0000 L CNN
-F 1 "R" V 5275 2625 50  0000 L CNN
+F 1 "10k" V 5275 2575 50  0000 L CNN
 F 2 "Resistor_THT:R_Axial_DIN0207_L6.3mm_D2.5mm_P10.16mm_Horizontal" V 5205 2650 50  0001 C CNN
 F 3 "~" H 5275 2650 50  0001 C CNN
@@
 P 5375 2650
 F 0 "R5" V 5325 2400 50  0000 L CNN
-F 1 "R" V 5375 2625 50  0000 L CNN
+F 1 "10k" V 5375 2575 50  0000 L CNN
 F 2 "Resistor_THT:R_Axial_DIN0207_L6.3mm_D2.5mm_P10.16mm_Horizontal" V 5305 2650 50  0001 C CNN
 F 3 "~" H 5375 2650 50  0001 C CNN
@@
 P 5475 2650
 F 0 "R6" V 5425 2400 50  0000 L CNN
-F 1 "R" V 5475 2625 50  0000 L CNN
+F 1 "10k" V 5475 2575 50  0000 L CNN
 F 2 "Resistor_THT:R_Axial_DIN0207_L6.3mm_D2.5mm_P10.16mm_Horizontal" V 5405 2650 50  0001 C CNN
 F 3 "~" H 5475 2650 50  0001 C CNN
@@
 P 5575 2650
 F 0 "R7" V 5525 2400 50  0000 L CNN
-F 1 "R" V 5575 2625 50  0000 L CNN
+F 1 "10k" V 5575 2575 50  0000 L CNN
 F 2 "Resistor_THT:R_Axial_DIN0207_L6.3mm_D2.5mm_P10.16mm_Horizontal" V 5505 2650 50  0001 C CNN
 F 3 "~" H 5575 2650 50  0001 C CNN
@@
 P 5675 2650
 F 0 "R8" V 5625 2400 50  0000 L CNN
-F 1 "R" V 5675 2625 50  0000 L CNN
+F 1 "10k" V 5675 2575 50  0000 L CNN
 F 2 "Resistor_THT:R_Axial_DIN0207_L6.3mm_D2.5mm_P10.16mm_Horizontal" V 5605 2650 50  0001 C CNN
 F 3 "~" H 5675 2650 50  0001 C CNN
@@
 	5675 2425 5675 2500
 Connection ~ 5575 2425
-Wire Notes Line
-	4850 2075 4850 2925
-Wire Notes Line
-	4850 2925 5800 2925
-Wire Notes Line
-	5800 2925 5800 2075
-Wire Notes Line
-	5800 2075 4850 2075
-Text Notes 4850 2050 0    50   ~ 0
-Need to check what the\nresistors needs to be.
+$Comp
+L Device:R R9
+U 1 1 6039E8EB
+P 9825 2650
+F 0 "R9" V 9775 2400 50  0000 L CNN
+F 1 "10k" V 9825 2575 50  0000 L CNN
+F 2 "Resistor_THT:R_Axial_DIN0207_L6.3mm_D2.5mm_P10.16mm_Horizontal" V 9755 2650 50  0001 C CNN
+F 3 "~" H 9825 2650 50  0001 C CNN
+	1    9825 2650
+	1    0    0    -1
+$EndComp
+Wire Wire Line
+	9825 2800 9825 3050
+Connection ~ 9825 3050
+$Comp
+L power:VCC #PWR02
+U 1 1 603A9B40
+P 9825 2500
+F 0 "#PWR02" H 9825 2350 50  0001 C CNN
+F 1 "VCC" H 9840 2673 50  0000 C CNN
+F 2 "" H 9825 2500 50  0001 C CNN
+F 3 "" H 9825 2500 50  0001 C CNN
+	1    9825 2500
+	1    0    0    -1
+$EndComp
 $EndSCHEMATC
