File: adapters/Amiga CD32/Amiga CD32.kicad_pcb (KiCad board)
At the start: 2 copper layers, 58.4 x 38.1 mm, 21 parts, among them J1 Port 1, J2 Port 2, J3 Sega Mega Drive, J4 START_SEL, M1 Mounting, M2 Mounting, M3 Mounting, M4 Mounting, SW1 START, U1 74LS157

Commit message: Layout done
Parts:
- removed J4: START_SEL, Connector_PinHeader_2.54mm:PinHeader_2x03_P2.54mm_Vertical
- removed R7, R8: 10k, Resistor_THT:R_Axial_DIN0207_L6.3mm_D2.5mm_P10.16mm_Horizontal
- added C2: 100nF, Capacitor_THT:C_Disc_D4.7mm_W2.5mm_P5.00mm, F.Cu at (117.5, 89.5)
- added C3: 47uF, Capacitor_THT:CP_Radial_D5.0mm_P2.00mm, F.Cu at (118.7, 82.5)
- added C4: 220pF, Capacitor_THT:C_Disc_D4.7mm_W2.5mm_P5.00mm, F.Cu at (168.3, 94.7)
- added C5: 220pF, Capacitor_THT:C_Disc_D4.7mm_W2.5mm_P5.00mm, F.Cu at (171.4, 81.9)
- added G***: LOGO, logo:c64_joykey, B.Cu at (148.1, 92.3)
- added L1: L, Inductor_THT:L_Axial_L6.6mm_D2.7mm_P10.16mm_Horizontal_Vishay_IM-2, F.Cu at (168.3, 81.9)
- added R10: 10k, resistor:R_Axial_DIN0207_L6.3mm_D2.5mm_P7.62mm_Horizontal, F.Cu at (153.7, 88.9)
- added R11: 10k, resistor:R_Axial_DIN0207_L6.3mm_D2.5mm_P10.16mm_Horizontal, F.Cu at (171.4, 99.7)
- added R12: 1k, resistor:R_Axial_DIN0207_L6.3mm_D2.5mm_P7.62mm_Horizontal, F.Cu at (134.6, 85.1)
- added R13: 100, resistor:R_Axial_DIN0207_L6.3mm_D2.5mm_P7.62mm_Horizontal, F.Cu at (149.9, 88.9)
- added R14: 10k, resistor:R_Axial_DIN0207_L6.3mm_D2.5mm_P10.16mm_Horizontal, F.Cu at (155.4, 99.7)
- added U2: 74LS165, Package_DIP:DIP-16_W7.62mm_Socket_LongPads, F.Cu at (120.7, 95.9)
- J3: value Sega Mega Drive -> Amiga CD32
- JP1: footprint Connector_PinHeader_2.54mm:PinHeader_1x02_P2.54mm_Vertical -> solder_bridge:bridge_r
- R1, R3, R4: footprint Resistor_THT:R_Axial_DIN0207_L6.3mm_D2.5mm_P10.16mm_Horizontal -> resistor:R_Axial_DIN0207_L6.3mm_D2.5mm_P10.16mm_Horizontal
- R2, R5, R6: footprint Resistor_THT:R_Axial_DIN0207_L6.3mm_D2.5mm_P10.16mm_Horizontal -> resistor:R_Axial_DIN0207_L6.3mm_D2.5mm_P7.62mm_Horizontal
- R9: value 10k -> 2k2; footprint Resistor_THT:R_Axial_DIN0207_L6.3mm_D2.5mm_P10.16mm_Horizontal -> resistor:R_Axial_DIN0207_L6.3mm_D2.5mm_P7.62mm_Horizontal
- SW1: value START -> PLAY
- U1: value 74LS157 -> 74LS125; footprint Package_DIP:DIP-16_W7.62mm_Socket_LongPads -> Package_DIP:DIP-14_W7.62mm_Socket_LongPads
- moved JP1 51.4 mm to (119.4, 103.5), turned to 270 degrees
- moved R6 27.9 mm to (146.1, 96.5), turned to 90 degrees
- moved R9 25.1 mm to (153.0, 85.1), turned to 180 degrees
- moved R5 22.9 mm to (131.4, 85.1)
- moved SW1 21.6 mm to (127.6, 78.7)
- moved R1 20.8 mm to (116.8, 99.7), turned to 0 degrees
- moved R2 11.2 mm to (142.2, 96.5), turned to 90 degrees
- moved R3 11.0 mm to (139.7, 99.7), turned to 180 degrees
- moved R4 10.9 mm to (152.4, 99.7), turned to 180 degrees
Connections:
- J1 pad 1: (no net) -> CD32_PLAY
- J1 pad 5: Net-(J1-Pad5) -> CD32_FF
- J1 pad 6: Net-(J1-Pad6) -> CD32_YEL
- J1 pad 9: Net-(J1-Pad9) -> CD32_REW
- J2 pad 1: /JK_UP -> UP
- J2 pad 2: /JK_DOWN -> DOWN
- J2 pad 3: /JK_LEFT -> LEFT
- J2 pad 4: /JK_RIGHT -> RIGHT
- J2 pad 5: /JK_FIRE3 -> CD32_GRN
- J2 pad 6: /JK_FIRE1 -> CD32_RED
- J2 pad 9: /JK_FIRE2 -> CD32_BLU
- J3 pad 1: /JK_UP -> UP
- J3 pad 2: /JK_DOWN -> DOWN
- J3 pad 3: /MD_LEFT -> LEFT
- J3 pad 4: /MD_RIGHT -> RIGHT
- J3 pad 5: VCC -> FIRE3
- J3 pad 6: /MD_B_A -> FIRE1
- J3 pad 7: /MD_SEL -> VCC
- J3 pad 9: /MD_C_START -> FIRE2
- JP1 pad 1: VCC -> Net-(J2-Pad7)
- JP1 pad 2: Net-(J2-Pad7) -> VCC
- R1 pad 2: /JK_UP -> CD32_RED
- R2 pad 2: /JK_DOWN -> CD32_GRN
- R3 pad 2: /JK_LEFT -> CD32_YEL
- R4 pad 2: /JK_RIGHT -> CD32_REW
- R5 pad 2: /JK_FIRE1 -> CD32_FF
- R6 pad 2: /JK_FIRE2 -> CD32_PLAY
- R9 pad 1: VCC -> Net-(R9-Pad1)
- R9 pad 2: /MD_SEL -> GND
- SW1 pad 2: /JK_START -> CD32_PLAY
- U1 pad 1: /MD_SEL -> FIRE3
- U1 pad 10: /JK_FIRE2 -> GND
- U1 pad 11: /JK_FIRE1 -> FIRE1
- U1 pad 12: /MD_C_START -> CD32_RED
- U1 pad 13: /JK_FIRE3 -> Net-(R9-Pad1)
- U1 pad 14: /JK_START -> VCC
- U1 pad 2: GND -> VCC
- U1 pad 3: /JK_LEFT -> Net-(R9-Pad1)
- U1 pad 4: /MD_LEFT -> Net-(R9-Pad1)
- U1 pad 6: /JK_RIGHT -> Net-(C4-Pad2)
- U1 pad 7: /MD_RIGHT -> GND
- U1 pad 8: GND -> Net-(L1-Pad2)
- U1 pad 9: /MD_B_A -> Net-(U1-Pad9)
Routing:
- net CD32_RED: track 0.00 -> 91.3 mm, vias 0 -> 2
- net VCC: track 111.1 -> 200.0 mm, vias 0 -> 2
- net FIRE1: track 0.00 -> 78.1 mm, vias 0 -> 2
- net /JK_START: track 76.1 -> 0.00 mm
- net Net-(C4-Pad2): track 0.00 -> 65.9 mm, vias 0 -> 1
- net CD32_GRN: track 0.00 -> 64.2 mm, vias 0 -> 1
- net CD32_PLAY: track 0.00 -> 57.7 mm, vias 0 -> 2
- net /MD_SEL: track 55.1 -> 0.00 mm, vias 1 -> 0
- net /JK_LEFT: track 53.9 -> 0.00 mm, vias 5 -> 0
- net /MD_B_A: track 51.2 -> 0.00 mm, vias 1 -> 0
- net /JK_FIRE3: track 48.6 -> 0.00 mm
- net /JK_FIRE1: track 47.1 -> 0.00 mm, vias 1 -> 0
- net /JK_UP: track 44.6 -> 0.00 mm
- net /JK_DOWN: track 41.9 -> 0.00 mm, vias 2 -> 0
- net CD32_FF: track 0.00 -> 40.6 mm
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Other:
- board text added: "Amiga CD32 github.com/tebl"
- board text removed: "(PORT 1)"
- board text removed: "FIRE1"
- board text removed: "FIRE2"
- board text removed: "FIRE3"
- board text removed: "J4 START_SEL"
- board text removed: "JP1 VCC_EN"
- board text removed: "P1 FIRE 1"
- board text removed: "Sega Mega Drive/Genesis (C64 JoyKEY Adapter) github.com/tebl"
