File: adapters/Amiga CD32/Amiga CD32.sch (KiCad schematic (older format))
At the start: 29 parts, among them J1 Port 1, J2 Port 2, J3 Amiga CD32, M1 Mounting, M2 Mounting, M3 Mounting, M4 Mounting, SW1 PLAY, U1 74LS125, U2 74LS165

Commit message: Layout done
Parts:
- R1, R11, R14, R3, R4: footprint Resistor_THT:R_Axial_DIN0207_L6.3mm_D2.5mm_P10.16mm_Horizontal -> resistor:R_Axial_DIN0207_L6.3mm_D2.5mm_P10.16mm_Horizontal
- R10, R12, R13, R2, R5, R6, R9: footprint Resistor_THT:R_Axial_DIN0207_L6.3mm_D2.5mm_P10.16mm_Horizontal -> resistor:R_Axial_DIN0207_L6.3mm_D2.5mm_P7.62mm_Horizontal
Changed lines of the file:
@@
 F 0 "R1" V 7125 1200 50  0000 L CNN
 F 1 "10k" V 7175 1425 50  0000 L CNN
-F 2 "Resistor_THT:R_Axial_DIN0207_L6.3mm_D2.5mm_P10.16mm_Horizontal" V 7105 1500 50  0001 C CNN
+F 2 "resistor:R_Axial_DIN0207_L6.3mm_D2.5mm_P10.16mm_Horizontal" V 7105 1500 50  0001 C CNN
 F 3 "~" H 7175 1500 50  0001 C CNN
 	1    7175 1500
@@
 F 0 "R9" V 4050 5200 50  0000 L CNN
 F 1 "2k2" V 4150 5175 50  0000 L CNN
-F 2 "Resistor_THT:R_Axial_DIN0207_L6.3mm_D2.5mm_P10.16mm_Horizontal" V 4080 5250 50  0001 C CNN
+F 2 "resistor:R_Axial_DIN0207_L6.3mm_D2.5mm_P7.62mm_Horizontal" V 4080 5250 50  0001 C CNN
 F 3 "~" H 4150 5250 50  0001 C CNN
 	1    4150 5250
@@
 F 0 "R10" V 4800 4300 50  0000 L CNN
 F 1 "10k" V 4900 4275 50  0000 L CNN
-F 2 "Resistor_THT:R_Axial_DIN0207_L6.3mm_D2.5mm_P10.16mm_Horizontal" V 4830 4350 50  0001 C CNN
+F 2 "resistor:R_Axial_DIN0207_L6.3mm_D2.5mm_P7.62mm_Horizontal" V 4830 4350 50  0001 C CNN
 F 3 "~" H 4900 4350 50  0001 C CNN
 	1    4900 4350
@@
 F 0 "R11" V 4800 5200 50  0000 L CNN
 F 1 "10k" V 4900 5175 50  0000 L CNN
-F 2 "Resistor_THT:R_Axial_DIN0207_L6.3mm_D2.5mm_P10.16mm_Horizontal" V 4830 5250 50  0001 C CNN
+F 2 "resistor:R_Axial_DIN0207_L6.3mm_D2.5mm_P10.16mm_Horizontal" V 4830 5250 50  0001 C CNN
 F 3 "~" H 4900 5250 50  0001 C CNN
 	1    4900 5250
@@
 F 0 "R13" V 5875 4175 50  0000 L CNN
 F 1 "100" V 5975 4175 50  0000 L CNN
-F 2 "Resistor_THT:R_Axial_DIN0207_L6.3mm_D2.5mm_P10.16mm_Horizontal" V 5905 4250 50  0001 C CNN
+F 2 "resistor:R_Axial_DIN0207_L6.3mm_D2.5mm_P7.62mm_Horizontal" V 5905 4250 50  0001 C CNN
 F 3 "~" H 5975 4250 50  0001 C CNN
 	1    5975 4250
@@
 F 0 "R12" V 5775 4175 50  0000 L CNN
 F 1 "1k" V 5875 4200 50  0000 L CNN
-F 2 "Resistor_THT:R_Axial_DIN0207_L6.3mm_D2.5mm_P10.16mm_Horizontal" V 5805 4250 50  0001 C CNN
+F 2 "resistor:R_Axial_DIN0207_L6.3mm_D2.5mm_P7.62mm_Horizontal" V 5805 4250 50  0001 C CNN
 F 3 "~" H 5875 4250 50  0001 C CNN
 	1    5875 4250
@@
 F 0 "R14" V 7225 1200 50  0000 L CNN
 F 1 "10k" V 7275 1425 50  0000 L CNN
-F 2 "Resistor_THT:R_Axial_DIN0207_L6.3mm_D2.5mm_P10.16mm_Horizontal" V 7205 1500 50  0001 C CNN
+F 2 "resistor:R_Axial_DIN0207_L6.3mm_D2.5mm_P10.16mm_Horizontal" V 7205 1500 50  0001 C CNN
 F 3 "~" H 7275 1500 50  0001 C CNN
 	1    7275 1500
@@
 F 0 "R2" V 7325 1200 50  0000 L CNN
 F 1 "10k" V 7375 1425 50  0000 L CNN
-F 2 "Resistor_THT:R_Axial_DIN0207_L6.3mm_D2.5mm_P10.16mm_Horizontal" V 7305 1500 50  0001 C CNN
+F 2 "resistor:R_Axial_DIN0207_L6.3mm_D2.5mm_P7.62mm_Horizontal" V 7305 1500 50  0001 C CNN
 F 3 "~" H 7375 1500 50  0001 C CNN
 	1    7375 1500
@@
 F 0 "R3" V 5250 1200 50  0000 L CNN
 F 1 "10k" V 5300 1425 50  0000 L CNN
-F 2 "Resistor_THT:R_Axial_DIN0207_L6.3mm_D2.5mm_P10.16mm_Horizontal" V 5230 1500 50  0001 C CNN
+F 2 "resistor:R_Axial_DIN0207_L6.3mm_D2.5mm_P10.16mm_Horizontal" V 5230 1500 50  0001 C CNN
 F 3 "~" H 5300 1500 50  0001 C CNN
 	1    5300 1500
@@
 F 0 "R4" V 5350 1200 50  0000 L CNN
 F 1 "10k" V 5400 1425 50  0000 L CNN
-F 2 "Resistor_THT:R_Axial_DIN0207_L6.3mm_D2.5mm_P10.16mm_Horizontal" V 5330 1500 50  0001 C CNN
+F 2 "resistor:R_Axial_DIN0207_L6.3mm_D2.5mm_P10.16mm_Horizontal" V 5330 1500 50  0001 C CNN
 F 3 "~" H 5400 1500 50  0001 C CNN
 	1    5400 1500
@@
 F 0 "R5" V 5450 1200 50  0000 L CNN
 F 1 "10k" V 5500 1425 50  0000 L CNN
-F 2 "Resistor_THT:R_Axial_DIN0207_L6.3mm_D2.5mm_P10.16mm_Horizontal" V 5430 1500 50  0001 C CNN
+F 2 "resistor:R_Axial_DIN0207_L6.3mm_D2.5mm_P7.62mm_Horizontal" V 5430 1500 50  0001 C CNN
 F 3 "~" H 5500 1500 50  0001 C CNN
 	1    5500 1500
@@
 F 0 "R6" V 5550 1200 50  0000 L CNN
 F 1 "10k" V 5600 1425 50  0000 L CNN
-F 2 "Resistor_THT:R_Axial_DIN0207_L6.3mm_D2.5mm_P10.16mm_Horizontal" V 5530 1500 50  0001 C CNN
+F 2 "resistor:R_Axial_DIN0207_L6.3mm_D2.5mm_P7.62mm_Horizontal" V 5530 1500 50  0001 C CNN
 F 3 "~" H 5600 1500 50  0001 C CNN
 	1    5600 1500
