File: C64 Joykey/C64 Joykey.sch (KiCad schematic (older format))
At the start: 57 parts, among them J1 Port_1, J2 Port_2, M1 Mounting, M2 Mounting, M3 Mounting, M4 Mounting, Q1 2N3904, SW1 FIRE1, SW2 FIRE2, SW3 FIRE3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

Commit message: Add discrete P1 switches
Parts:
- added SW10: P1_FIRE2, Button_Switch_THT:SW_Tactile_SPST_Angled_PTS645Vx31-2LFS, symbol Switch:SW_Push
- added SW11: P1_FIRE3, Button_Switch_THT:SW_Tactile_SPST_Angled_PTS645Vx31-2LFS, symbol Switch:SW_Push
- added SW9: P1_FIRE1, Button_Switch_THT:SW_Tactile_SPST_Angled_PTS645Vx31-2LFS, symbol Switch:SW_Push
- SW1: value FIRE1 -> P2_FIRE1; symbol sw_keyboard:SW_Keyboard -> Switch:SW_Push
- SW2: value FIRE2 -> P2_FIRE2; symbol sw_keyboard:SW_Keyboard -> Switch:SW_Push
- SW3: value FIRE3 -> P2_FIRE3; symbol sw_keyboard:SW_Keyboard -> Switch:SW_Push
- SW4, SW5, SW6, SW7: symbol sw_keyboard:SW_Keyboard -> Switch:SW_Push
Connections:
- net FIRE2_POL: now also SW2.1, SW10.1; no longer SW2.2
- net FIRE3_POL: now also SW3.1, SW11.1; no longer SW3.2
- net GND: now also SW1.1, SW4.1, SW5.1, SW6.1, SW7.1, SW9.1; no longer SW1.2, SW4.2, SW5.2, SW6.2, SW7.2
- net P1_FIRE1: now also SW9.2
- net P2_DOWN: now also SW5.2; no longer SW5.1
- net P2_LEFT: now also SW6.2; no longer SW6.1
- net P2_RIGHT: now also SW7.2; no longer SW7.1
- net P2_UP: now also SW4.2; no longer SW4.1
- net at JP4.1, R17.2: now also SW1.2; no longer SW1.1
- net at JP6.1, R16.2: now also SW2.2; no longer SW2.1
- net at JP3.2 (C), R15.2: now also SW3.2; no longer SW3.1
- net P1_FIRE3: now reaches J1.5 (Pin_5)
- net P1_FIRE3: now also SW11.2
- net P1_FIRE2: now reaches J1.9 (Pin_9)
- net P1_FIRE2: now also SW10.2
- no-connect marks 12 -> 10
Other:
- note added: "DIRECTIONS:"
- note added: "FIRE 1:"
- note added: "FIRE 2:"
- note added: "FIRE 3:"
- note added: "JP1 (FIRE2 polarity):\n1-2 C64 (POTX)\nN/C Other system\n\nWARNING: Read documentation for\ndetails, especially if not a C64."
- note added: "JP2 (FIRE3 polarity):\n1-2 C64 (POTY)\nN/C Other system\n\nWARNING: Read documentation for\ndetails, especially if not a C64."
- note added: "Linking 1-2 will light PWR LED\npermanently, 2-3 allows Arduino\nto take control of it instead."
- note added: "Underglow LEDs:"
- note removed: "JP1 (FIRE2 polarity):\n1-2 C64 (POTX)\nN/C Other system\n\nRead documentation for\ndetails if not C64."
- note removed: "JP2 (FIRE3 polarity):\n1-2 C64 (POTY)\nN/C Other system\n\nRead documentation for\ndetails if not C64.\n"
- note removed: "Linking 1-2 will light PWR LED\npermanently, 2-3 enables\nArduino to control it."
- moved on the sheet: A1, D1, D10, D11, D2, D3, D4, D5, D6, D7, D8, D9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

Commit message: Route new tracks and export gerbers
Parts:
- SW1, SW10, SW11, SW2, SW3, SW4, SW5, SW6, SW7, SW9: symbol Switch:SW_Push -> sw_push:SW_Push
Connections:
- net FIRE2_POL: now also SW10.2, SW2.2; no longer SW10.1, SW2.1
- net FIRE3_POL: now also SW11.2, SW3.2; no longer SW11.1, SW3.1
- net GND: now also SW1.2, SW4.2, SW5.2, SW6.2, SW7.2, SW9.2; no longer SW1.1, SW4.1, SW5.1, SW6.1, SW7.1, SW9.1
- net P1_FIRE1: now also SW9.1; no longer SW9.2
- net P1_FIRE2: now also SW10.1; no longer SW10.2
- net P1_FIRE3: now also SW11.1; no longer SW11.2
- net P2_DOWN: now also SW5.1; no longer SW5.2
- net P2_LEFT: now also SW6.1; no longer SW6.2
- net P2_RIGHT: now also SW7.1; no longer SW7.2
- net P2_UP: now also SW4.1; no longer SW4.2
- net at JP4.1, R17.2: now also SW1.1; no longer SW1.2
- net at JP6.1, R16.2: now also SW2.1; no longer SW2.2
- net at JP3.2 (C), R15.2: now also SW3.1; no longer SW3.2
Other:
- note added: "As is common, but definitely not always, on the\nCommodore 64, port 2 is the main controller port.\nPort 1 is simply used for additional fire buttons, at\nthe moment it does not include direction signals\n(this is by design).\n\nPay particular attention to the polarity settings\nfor the switches, these need to be set correctly\nin order to avoid damaging the system (this will\naffect both ports).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"
- note added: "OUTPUT:"
- moved on the sheet: A1, D1, D2, D3, D4, J1, J2, JP5, JP8, JP9, R14, R15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

Commit message: Add missing CD32 button
Parts:
- added SW12: P1_FIRE4, Button_Switch_THT:SW_Tactile_SPST_Angled_PTS645Vx31-2LFS, symbol sw_push:SW_Push
- JP4: footprint Connector_PinHeader_2.54mm:PinHeader_1x02_P2.54mm_Vertical -> solder_bridge:bridge
- JP6: footprint Connector_PinHeader_2.54mm:PinHeader_1x02_P2.54mm_Vertical -> solder_bridge:bridge_r
Connections:
- net GND: now also SW12.2
- net P1_FIRE4: now reaches J1.1 (Pin_1)
- net P1_FIRE4: now also SW12.1
- no-connect marks 10 -> 9
Other:
- moved on the sheet: SW4, SW5, SW6, SW7
Changed lines of the file:
@@
 	1    0    0    -1
 $EndComp
-NoConn ~ 11075 3175
 NoConn ~ 11075 3275
 NoConn ~ 11075 3375
@@
 L sw_push:SW_Push SW4
 U 1 1 5FB7E128
-P 1625 3225
-F 0 "SW4" H 1525 3325 50  0000 C CNN
-F 1 "UP" H 1625 3150 50  0000 C CNN
-F 2 "Button_Switch_Keyboard:SW_Cherry_MX_1.00u_PCB" H 1625 3425 50  0001 C CNN
-F 3 "" H 1625 3425 50  0001 C CNN
-	1    1625 3225
+P 1650 2125
+F 0 "SW4" H 1550 2225 50  0000 C CNN
+F 1 "UP" H 1650 2050 50  0000 C CNN
+F 2 "Button_Switch_Keyboard:SW_Cherry_MX_1.00u_PCB" H 1650 2325 50  0001 C CNN
+F 3 "" H 1650 2325 50  0001 C CNN
+	1    1650 2125
 	1    0    0    -1
 $EndComp
@@
 L sw_push:SW_Push SW5
 U 1 1 5FB7E12E
-P 1625 3750
-F 0 "SW5" H 1525 3850 50  0000 C CNN
-F 1 "DOWN" H 1625 3675 50  0000 C CNN
-F 2 "Button_Switch_Keyboard:SW_Cherry_MX_1.00u_PCB" H 1625 3950 50  0001 C CNN
-F 3 "" H 1625 3950 50  0001 C CNN
-	1    1625 3750
+P 1650 2650
+F 0 "SW5" H 1550 2750 50  0000 C CNN
+F 1 "DOWN" H 1650 2575 50  0000 C CNN
+F 2 "Button_Switch_Keyboard:SW_Cherry_MX_1.00u_PCB" H 1650 2850 50  0001 C CNN
+F 3 "" H 1650 2850 50  0001 C CNN
+	1    1650 2650
 	1    0    0    -1
 $EndComp
@@
 L sw_push:SW_Push SW6
 U 1 1 5FB7E134
-P 1625 4275
-F 0 "SW6" H 1525 4375 50  0000 C CNN
-F 1 "LEFT" H 1625 4200 50  0000 C CNN
-F 2 "Button_Switch_Keyboard:SW_Cherry_MX_1.00u_PCB" H 1625 4475 50  0001 C CNN
-F 3 "" H 1625 4475 50  0001 C CNN
-	1    1625 4275
+P 1650 3175
+F 0 "SW6" H 1550 3275 50  0000 C CNN
+F 1 "LEFT" H 1650 3100 50  0000 C CNN
+F 2 "Button_Switch_Keyboard:SW_Cherry_MX_1.00u_PCB" H 1650 3375 50  0001 C CNN
+F 3 "" H 1650 3375 50  0001 C CNN
+	1    1650 3175
 	1    0    0    -1
 $EndComp
@@
 L power:GND #PWR04
 U 1 1 5FB7E13A
-P 1275 5325
-F 0 "#PWR04" H 1275 5075 50  0001 C CNN
-F 1 "GND" H 1280 5152 50  0000 C CNN
-F 2 "" H 1275 5325 50  0001 C CNN
-F 3 "" H 1275 5325 50  0001 C CNN
-	1    1275 5325
+P 1300 3775
+F 0 "#PWR04" H 1300 3525 50  0001 C CNN
+F 1 "GND" H 1305 3602 50  0000 C CNN
+F 2 "" H 1300 3775 50  0001 C CNN
+F 3 "" H 1300 3775 50  0001 C CNN
+	1    1300 3775
 	1    0    0    -1
 $EndComp
@@
 L sw_push:SW_Push SW7
 U 1 1 5FB81454
-P 1625 4800
-F 0 "SW7" H 1525 4900 50  0000 C CNN
-F 1 "RIGHT" H 1625 4725 50  0000 C CNN
-F 2 "Button_Switch_Keyboard:SW_Cherry_MX_1.00u_PCB" H 1625 5000 50  0001 C CNN
-F 3 "" H 1625 5000 50  0001 C CNN
-	1    1625 4800
-	1    0    0    -1
-$EndComp
-Text GLabel 1900 3225 2    50   Output ~ 0
+P 1650 3700
+F 0 "SW7" H 1550 3800 50  0000 C CNN
+F 1 "RIGHT" H 1650 3625 50  0000 C CNN
+F 2 "Button_Switch_Keyboard:SW_Cherry_MX_1.00u_PCB" H 1650 3900 50  0001 C CNN
+F 3 "" H 1650 3900 50  0001 C CNN
+	1    1650 3700
+	1    0    0    -1
+$EndComp
+Text GLabel 1925 2125 2    50   Output ~ 0
 P2_UP
-Text GLabel 1900 4275 2    50   Output ~ 0
+Text GLabel 1925 3175 2    50   Output ~ 0
 P2_LEFT
-Text GLabel 1900 3750 2    50   Output ~ 0
+Text GLabel 1925 2650 2    50   Output ~ 0
 P2_DOWN
-Text GLabel 1900 4800 2    50   Output ~ 0
+Text GLabel 1925 3700 2    50   Output ~ 0
 P2_RIGHT
 Text GLabel 5450 3800 2    50   Output ~ 0
@@
 F 0 "JP6" H 5175 3975 50  0000 C CNN
 F 1 "DEFAULT_FW" H 5175 3900 50  0000 C CNN
-F 2 "Connector_PinHeader_2.54mm:PinHeader_1x02_P2.54mm_Vertical" H 5175 3800 50  0001 C CNN
+F 2 "solder_bridge:bridge_r" H 5175 3800 50  0001 C CNN
 F 3 "~" H 5175 3800 50  0001 C CNN
 	1    5175 3800
@@
 F 0 "JP4" H 5175 2500 50  0000 C CNN
 F 1 "DEFAULT_FW" H 5175 2425 50  0000 C CNN
-F 2 "Connector_PinHeader_2.54mm:PinHeader_1x02_P2.54mm_Vertical" H 5175 2325 50  0001 C CNN
+F 2 "solder_bridge:bridge" H 5175 2325 50  0001 C CNN
 F 3 "~" H 5175 2325 50  0001 C CNN
 	1    5175 2325
@@
 	825  1750 2600 1750
 Wire Wire Line
-	1825 3225 1900 3225
-Connection ~ 1275 3750
-Wire Wire Line
-	1275 3225 1275 3750
-Wire Wire Line
-	1275 3750 1275 4275
-Wire Wire Line
-	1275 3225 1425 3225
-Wire Wire Line
-	1275 3750 1425 3750
-Wire Wire Line
-	1900 3750 1825 3750
-Wire Wire Line
-	1275 4275 1425 4275
-Connection ~ 1275 4275
-Wire Wire Line
-	1275 4275 1275 4800
-Wire Wire Line
-	1275 4800 1425 4800
-Connection ~ 1275 4800
-Wire Wire Line
-	1900 4800 1825 4800
-Wire Wire Line
-	1825 4275 1900 4275
-Wire Wire Line
-	1275 4800 1275 5325
+	1850 2125 1925 2125
+Connection ~ 1300 2650
+Wire Wire Line
+	1300 2125 1300 2650
+Wire Wire Line
+	1300 2650 1300 3175
+Wire Wire Line
+	1300 2125 1450 2125
+Wire Wire Line
+	1300 2650 1450 2650
+Wire Wire Line
+	1925 2650 1850 2650
+Wire Wire Line
+	1300 3175 1450 3175
+Connection ~ 1300 3175
+Wire Wire Line
+	1300 3175 1300 3700
+Wire Wire Line
+	1300 3700 1450 3700
+Wire Wire Line
+	1925 3700 1850 3700
+Wire Wire Line
+	1850 3175 1925 3175
 Text Notes 825  1725 0    98   ~ 0
 DIRECTIONS:
@@
 Text Notes 13600 3075 0    50   ~ 0
 As is common, but definitely not always, on the\nCommodore 64, port 2 is the main controller port.\nPort 1 is simply used for additional fire buttons, at\nthe moment it does not include direction signals\n(this is by design).\n\nPay particular attention to the polarity settings\nfor the switches, these need to be set correctly\nin order to avoid damaging the system (this will\naffect both ports). An adapter designed for a\nspecific system will usually denote this setting.
+Text GLabel 10925 3175 0    50   Input ~ 0
+P1_FIRE4
+Wire Wire Line
+	10925 3175 11075 3175
+Text GLabel 1925 5125 2    50   Output ~ 0
+P1_FIRE4
+$Comp
+L sw_push:SW_Push SW12
+U 1 1 62D9D03F
+P 1650 5125
+F 0 "SW12" H 1550 5225 50  0000 C CNN
+F 1 "P1_FIRE4" H 1650 5050 50  0000 C CNN
+F 2 "Button_Switch_THT:SW_Tactile_SPST_Angled_PTS645Vx31-2LFS" H 1650 5325 50  0001 C CNN
+F 3 "" H 1650 5325 50  0001 C CNN
+	1    1650 5125
+	1    0    0    -1
+$EndComp
+Wire Wire Line
+	1850 5125 1925 5125
+Wire Wire Line
+	1450 5125 1300 5125
+Wire Wire Line
+	1300 3775 1300 3700
+Connection ~ 1300 3700
+$Comp
+L power:GND #PWR0107
+U 1 1 62DF21A8
+P 1300 5200
+F 0 "#PWR0107" H 1300 4950 50  0001 C CNN
+F 1 "GND" H 1305 5027 50  0000 C CNN
+F 2 "" H 1300 5200 50  0001 C CNN
+F 3 "" H 1300 5200 50  0001 C CNN
+	1    1300 5200
+	1    0    0    -1
+$EndComp
+Wire Wire Line
+	1300 5200 1300 5125
 $EndSCHEMATC

Commit message: Change recommended diode type to 1n5819 for lower voltage drop
Parts:
- D3: value 1n4001 -> 1n5819; symbol Device:D -> Diode:1N5819
Changed lines of the file:
@@
 	5275 3800 5450 3800
 $Comp
-L Device:D D3
+L Diode:1N5819 D3
 U 1 1 5FCFF93E
 P 13175 2475
 F 0 "D3" H 13175 2259 50  0000 C CNN
-F 1 "1n4001" H 13175 2350 50  0000 C CNN
+F 1 "1n5819" H 13175 2350 50  0000 C CNN
 F 2 "Diodes_THT:D_DO-41_SOD81_P10.16mm_Horizontal" H 13175 2475 50  0001 C CNN
 F 3 "~" H 13175 2475 50  0001 C CNN
