File: C64 Joykey 2040/Output.kicad_sch (KiCad schematic)
At the start: 4 parts, among them J1 Port_1, J2 Port_2

Commit message: First layout drafted
Other:
- note added: "The jumper VCC_EN is to enable the computer to power up the C64 JoyKEY, a diode has been added to ensure that other direction doesn't happen. Power is always routed through to APWR, but this is only used in order to provide power to the adapters themselves. Not sure if I'll ever need it, but if I have it - then I have it."
- note removed: "The jumper VCC_EN is to enable the computer to power up the C64 JoyKEY, a diode has been added to ensure that other direction doesn't happen. Power is always routed through to APWR, this is only used in order to provide power to the adapters themselves. Not sure if I'll ever need it, but if I have it - then I'll have it."
Changed lines of the file:
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@@
 		)
 	)
-	(text "The jumper VCC_EN is to enable the computer to\npower up the C64 JoyKEY, a diode has been added\nto ensure that other direction doesn't happen.\n\nPower is always routed through to APWR, this is\nonly used in order to provide power to the\nadapters themselves. Not sure if I'll ever need\nit, but if I have it - then I'll have it."
+	(text "The jumper VCC_EN is to enable the computer to\npower up the C64 JoyKEY, a diode has been added\nto ensure that other direction doesn't happen.\n\nPower is always routed through to APWR, but this\nis only used in order to provide power to the\nadapters themselves. Not sure if I'll ever need\nit, but if I have it - then I have it."
 		(exclude_from_sim no)
 		(at 199.39 83.82 0)
