File: C64 Joykey 2040/C64 Joykey 2040.kicad_sch (KiCad schematic)
At the start: 22 parts, among them J4 Expansion, M1 Mounting, M2 Mounting, M3 Mounting, M4 Mounting, U1 RP2040-Zero

Commit message: Change expansion header to JST XH, but in a right-angle variant
Parts:
- J4: footprint Connector_PinHeader_2.54mm:PinHeader_1x04_P2.54mm_Vertical -> JST_XH_Right_Angle:JST_XH_B4B-XH-A_1x04_P2.50mm_Right_Angle
Changed lines of the file:
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@@
 			)
 		)
-		(property "Footprint" "Connector_PinHeader_2.54mm:PinHeader_1x04_P2.54mm_Vertical"
+		(property "Footprint" "JST_XH_Right_Angle:JST_XH_B4B-XH-A_1x04_P2.50mm_Right_Angle"
 			(at 252.73 138.43 0)
 			(effects
