File: Adapter 9 from 2040/Display.kicad_sch (KiCad schematic)
At the start: 3 parts, among them IC1 0.96_I2C_OLED

Commit message: Slight tweaks
Parts:
- renumbered JP3 to JP2, JP2 to JP3
Changed lines of the file:
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@@
 		(on_board yes)
 		(dnp no)
-		(property "Reference" "JP3"
+		(property "Reference" "JP2"
 			(at 163.0172 82.6516 90)
 			(effects
@@
 			(project "Adapter 9 from 2040"
 				(path "/1673ead5-026d-4add-8d8b-47a838e01efc/2fa2432a-52d4-42db-b1d9-b3c408329551"
-					(reference "JP3")
+					(reference "JP2")
 					(unit 1)
 				)
@@
 		(on_board yes)
 		(dnp no)
-		(property "Reference" "JP2"
+		(property "Reference" "JP3"
 			(at 144.3228 82.6516 90)
 			(effects
@@
 			(project "Adapter 9 from 2040"
 				(path "/1673ead5-026d-4add-8d8b-47a838e01efc/2fa2432a-52d4-42db-b1d9-b3c408329551"
-					(reference "JP2")
+					(reference "JP3")
 					(unit 1)
 				)
