File: Adapter 9 from 2040/Adapter 9 from 2040.kicad_pcb (KiCad board)
At the start: 2 copper layers, 70.7 x 46.7 mm, 21 parts, among them IC1 0.96_I2C_OLED, J1 Atari, M1 Mounting, M2 Mounting, M3 Mounting, M4 Mounting, SW1 S1, SW2 S2, SW3 L1, SW4 R1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

Commit message: Slight tweaks
Parts:
- JP2: value P2_VCC -> P1_GND
- JP3: value P1_GND -> P2_VCC
- moved JP2 3.18 mm to (191.1, 116.8), turned to 90 degrees
- moved JP3 3.18 mm to (194.3, 116.8), turned to -90 degrees
Connections:
- JP2 pad 1: +3V3 -> GND
- JP2 pad 2: Net-(IC1-VCC) -> Net-(IC1-GND)
- JP2 pad 3: GND -> +3V3
- JP3 pad 1: GND -> +3V3
- JP3 pad 2: Net-(IC1-GND) -> Net-(IC1-VCC)
- JP3 pad 3: +3V3 -> GND
Other:
- board text added: "JP2"
- board text added: "JP3"
- board text added: "SCL"
- board text added: "SDA"

Commit message: PCBway order number placeholder
Other:
- board text added: "WayWayWay"
Changed lines of the file:
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@@
+		)
+	)
+	(gr_text "WayWayWay"
+		(at 160.169698 118.1565 270)
+		(layer "F.SilkS")
+		(effects
+			(font
+				(size 0.8 0.8)
+				(thickness 0.1)
+			)
 		)
 	)
